File: converterboard/converterboard.kicad_pcb (KiCad board)
At the start: 2 copper layers, 39 x 30 mm, 17 parts, among them CON1 FPC_6POS, J1 USB_B_Micro, J2 Conn_02x10_Odd_Even, J3 Conn_01x04, U1 FT232RL, U2 TXB0108PWR

Commit message: HW rev 1+2
Parts:
- removed J1: USB_B_Micro, Connector_USB:USB_Micro-B_Molex_47346-0001
- removed L1: Ferrite_Bead_Small, Inductor_SMD:L_0603_1608Metric
- added J4: USB_C_Receptacle, athir:DX07S024JJ, F.Cu at (195.8, 113.9)
- added L2: Ferrite_Bead_Small, Inductor_SMD:L_0603_1608Metric, F.Cu at (188.2, 117.2)
- R2, R3: value R_Small -> 100
- moved J2 1.25 mm to (173.5, 123.8)
Connections:
- C1 pad 1: Net-(C1-Pad1) -> VBUS
Routing:
- net Net-(J4-PadA4): track 0.00 -> 13.7 mm
- net VBUS: track 32.9 -> 43.7 mm
- net Net-(C1-Pad1): track 9.41 -> 0.00 mm
- net /D+: track 11.3 -> 18.1 mm, vias 2 -> 3
- net /D-: track 12.7 -> 16.0 mm
- net VCC: track 44.7 -> 42.5 mm
- net /SWDIO: track 41.4 -> 40.0 mm
- net /MCU_RESET: track 58.7 -> 57.6 mm
- net /SWCLK: track 47.8 -> 47.1 mm
- net GND: vias 60 -> 108
- net (no net): vias 0 -> 2
Other:
- board size 39 x 30 mm -> 43.8 x 30 mm
- board text added: "- RX TX +"
- board text added: "Converter board Rev. 2 - 1912"

Commit message: HW rev 3 - Sorry future me.. dunno what I changed. But it might be for the SC2???
Parts:
- C2: footprint Capacitor_THT:CP_Radial_D5.0mm_P2.00mm -> Capacitor_SMD:C_0805_2012Metric
- moved C3 1.35 mm to (179.0, 116.5)
- moved C2 0.50 mm to (181.8, 115.5), turned to 0 degrees
Connections:
- U1 pad 1: /RXD -> /TXD
- U1 pad 5: /TXD -> /RXD
Routing:
- net /RXD: track 13.0 -> 8.41 mm
- net /TXD: track 6.54 -> 10.1 mm, vias 0 -> 2
- net +3V3: track 11.1 -> 8.21 mm
- net GND: vias 108 -> 110
Other:
- board text added: "Converter board Rev. 3 - 1922"
- board text removed: "Converter board Rev. 2 - 1912"
